Commit message: Refactor code structure and remove redundant sections for improved readability and maintainability

File: taller1/taller2_ras/install/ros_package/share/ros_package/urdf/pepper.urdf (robot description, URDF)
Before this commit: robot pepper, 3 links, 2 joints
Links:
- link torso: geometry collision mesh filename=package://ros_package/urdf/mesh/chest.stl scale=1 1 1; visual mesh filename=package://ros_package/urdf/mesh/chest.stl scale=1 1 1

File: taller1/taller2_ras/src/ros_package/urdf/pepper.urdf (robot description, URDF)
Before this commit: robot pepper, 3 links, 2 joints
Links:
- added link base; visual mesh filename=package://ros_package/urdf/mesh/base.stl scale=1 1 1
- link base_link: geometry 
- link torso: geometry collision mesh filename=package://ros_package/urdf/mesh/chest.stl scale=1 1 1; visual mesh filename=package://ros_package/urdf/mesh/chest.stl scale=1 1 1

Commit message: .

File: taller1/taller2_ras/install/ros_package/share/ros_package/urdf/pepper.urdf (robot description, URDF)
Before this commit: robot pepper, 3 links, 2 joints
Links:
- removed link base_link
- removed link brazo
- added link base; collision mesh filename=package://ros_package/urdf/mesh/base.stl scale=1 1 1; visual mesh filename=package://ros_package/urdf/mesh/base.stl scale=1 1 1
- added link lower_body; collision mesh filename=package://ros_package/urdf/mesh/lower_body.stl scale=1 1 1; visual mesh filename=package://ros_package/urdf/mesh/lower_body.stl scale=1 1 1
Joints:
- removed joint base_to_torso
- removed joint torso_to_brazo
- added joint base_to_lower_body: type revolute, parent base, child lower_body, origin xyz=0 0 0.32 rpy=0 0 0, axis 1 0 0, limit lower=-0.25 upper=0.25 effort=1000 velocity=0.5
- added joint lower_body_to_torso: type fixed, parent lower_body, child torso, origin xyz=0 0.02 0.39 rpy=0 0 0

File: taller1/taller2_ras/src/ros_package/urdf/pepper.urdf (robot description, URDF)
Before this commit: robot pepper, 4 links, 2 joints
Links:
- removed link base_link
- removed link brazo
- added link lower_body; collision mesh filename=package://ros_package/urdf/mesh/lower_body.stl scale=1 1 1; visual mesh filename=package://ros_package/urdf/mesh/lower_body.stl scale=1 1 1
- link base: geometry collision mesh filename=package://ros_package/urdf/mesh/base.stl scale=1 1 1; visual mesh filename=package://ros_package/urdf/mesh/base.stl scale=1 1 1
Joints:
- removed joint base_to_torso
- removed joint torso_to_brazo
- added joint base_to_lower_body: type revolute, parent base, child lower_body, origin xyz=0 0 0.32 rpy=0 0 0, axis 1 0 0, limit lower=-0.25 upper=0.25 effort=1000 velocity=0.5
- added joint lower_body_to_torso: type fixed, parent lower_body, child torso, origin xyz=0 0.02 0.39 rpy=0 0 0
